Commit message: add mapa1, refactor parâmetros do controller

File: src/mec_description/urdf/mec_core.xacro (robot description, xacro)
@@ -21,4 +21,9 @@
         <child link="base_link"/>
         <origin xyz="0 0 0.07" rpy="0 0 0"/>
+    </joint>
+    <joint name="base_footprint_to_base_link_joint" type="fixed">
+        <parent link="base_footprint"/>
+        <child link="base_link"/>
+        <origin xyz="0.0 0.0 0.08"/>
     </joint>
     <!-- Chassis -->
